File: Thermostat.sch (KiCad schematic (older format))
At the start: 21 parts, among them P1 PWR, P2 NTC probe 8K, P3 HEATER, U1 LM358, U2 MOC3063M, U3 TRIAC

Commit message: Updated schematic
Parts:
- removed D1: 1N4001, symbol D
- removed R2: 22K, symbol R
- added D1: Diode_Bridge, symbol Diode_Bridge
- C1: value 680n -> 470n; footprint (none) -> Capacitors_ThroughHole:C_Rect_L13.5mm_W5.0mm_P10.00mm_FKS3_FKP3_MKS4
- C2: renamed from C3; value 100u -> 220u
- C3: renamed from C2; footprint (none) -> Capacitors_SMD:C_1206_HandSoldering
- P3: renamed from P2; value NTC probe 8K -> NTC probe 10K
- R1: value 4K7K -> 1K/2W
- RV1: value 1K -> 2K2
- renumbered P3 to P1, P1 to P2, R3 to R2, R4 to R3, R5 to R4, R6 to R5, R7 to R6, R8 to R7
Connections:
- net GND: now also D1.1 (-); no longer P2.1 (P1), R7.2, U3.1
- net at C2.1, C3.1, D2.1 (K)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: now also D1.3 (+)
- net at R6.1, U3.3: now also R7.2; no longer R7.1
- net at C1.1: now also D1.4
- new net: D1.2, P2.1 (P1), R7.1, U3.1
Other:
- moved on the sheet: C1, C2, C3, D2, D3, P1, P2, P3, R1, R2, R3, R4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

Commit message: Started the PCB
Parts:
- C2: footprint (none) -> Capacitors_ThroughHole:CP_Radial_D7.5mm_P2.50mm
- D1: footprint (none) -> Diodes_ThroughHole:Diode_Bridge_15.7x15.7
- D2: footprint (none) -> Diodes_ThroughHole:D_T-1_P5.08mm_Horizontal
- D3, P3: footprint (none) -> Socket_Strips:Socket_Strip_Straight_1x02_Pitch2.54mm
- P1, P2: footprint (none) -> Socket_Strips:Socket_Strip_Angled_1x02_Pitch2.54mm
- R1: footprint (none) -> Resistors_ThroughHole:R_Axial_DIN0207_L6.3mm_D2.5mm_P10.16mm_Horizontal
- R2, R3, R4, R6, R7: footprint (none) -> Resistors_SMD:R_1206_HandSoldering
- R5: value 220R -> 1K; footprint (none) -> Resistors_SMD:R_1206_HandSoldering
- RV1: footprint (none) -> Potentiometers:Potentiometer_Piher_PC-16_Single_Horizontal
- U1: footprint (none) -> Housings_DIP:DIP-8_W7.62mm
- U2: footprint DIP-6 -> Housings_DIP:DIP-6_W7.62mm
- U3: footprint (none) -> Socket_Strips:Socket_Strip_Straight_1x03_Pitch2.54mm
Connections:
- net GND: no longer names the net of C2.2, C3.2, D1.1 (-), D2.2 (A), P3.1 (P1), R4.2, U1.4 (V-), U2.2
Changed lines of the file:
@@
 F 0 "U1" H 7350 3800 50  0000 L CNN
 F 1 "LM358" H 7350 3350 50  0000 L CNN
-F 2 "" H 7400 3600 50  0001 C CNN
+F 2 "Housings_DIP:DIP-8_W7.62mm" H 7400 3600 50  0001 C CNN
 F 3 "" H 7400 3600 50  0000 C CNN
 	1    7400 3600
@@
 F 0 "R2" V 6380 3350 50  0000 C CNN
 F 1 "10K" V 6300 3350 50  0000 C CNN
-F 2 "" V 6230 3350 50  0001 C CNN
+F 2 "Resistors_SMD:R_1206_HandSoldering" V 6230 3350 50  0001 C CNN
 F 3 "" H 6300 3350 50  0000 C CNN
 	1    6300 3350
@@
 F 0 "R3" V 6780 3150 50  0000 C CNN
 F 1 "10K" V 6700 3150 50  0000 C CNN
-F 2 "" V 6630 3150 50  0001 C CNN
+F 2 "Resistors_SMD:R_1206_HandSoldering" V 6630 3150 50  0001 C CNN
 F 3 "" H 6700 3150 50  0000 C CNN
 	1    6700 3150
@@
 F 0 "R4" V 6780 4300 50  0000 C CNN
 F 1 "6K8" V 6700 4300 50  0000 C CNN
-F 2 "" V 6630 4300 50  0001 C CNN
+F 2 "Resistors_SMD:R_1206_HandSoldering" V 6630 4300 50  0001 C CNN
 F 3 "" H 6700 4300 50  0000 C CNN
 	1    6700 4300
@@
 F 0 "RV1" H 6700 3420 50  0000 C CNN
 F 1 "2K2" H 6700 3500 50  0000 C CNN
-F 2 "" H 6700 3500 50  0001 C CNN
+F 2 "Potentiometers:Potentiometer_Piher_PC-16_Single_Horizontal" H 6700 3500 50  0001 C CNN
 F 3 "" H 6700 3500 50  0000 C CNN
 	1    6700 3500
@@
 F 0 "U2" H 8600 3900 50  0000 L CNN
 F 1 "MOC3063M" H 8800 3900 50  0000 L CNN
-F 2 "DIP-6" H 8600 3500 50  0000 L CIN
+F 2 "Housings_DIP:DIP-6_W7.62mm" H 8600 3500 50  0000 L CIN
 F 3 "" H 8790 3700 50  0000 L CNN
 	1    8800 3700
@@
 P 7900 3600
 F 0 "R5" V 7980 3600 50  0000 C CNN
-F 1 "220R" V 7900 3600 50  0000 C CNN
-F 2 "" V 7830 3600 50  0001 C CNN
+F 1 "1K" V 7900 3600 50  0000 C CNN
+F 2 "Resistors_SMD:R_1206_HandSoldering" V 7830 3600 50  0001 C CNN
 F 3 "" H 7900 3600 50  0000 C CNN
 	1    7900 3600
@@
 F 0 "D2" H 4400 3550 50  0000 C CNN
 F 1 "ZD12V" H 4400 3350 50  0000 C CNN
-F 2 "" H 4400 3450 50  0001 C CNN
+F 2 "Diodes_ThroughHole:D_T-1_P5.08mm_Horizontal" H 4400 3450 50  0001 C CNN
 F 3 "" H 4400 3450 50  0000 C CNN
 	1    4400 3450
 	0    1    1    0
-$EndComp
-$Comp
-L GND #PWR01
-U 1 1 58D1B486
-P 6300 4650
-F 0 "#PWR01" H 6300 4400 50  0001 C CNN
-F 1 "GND" H 6300 4500 50  0000 C CNN
-F 2 "" H 6300 4650 50  0000 C CNN
-F 3 "" H 6300 4650 50  0000 C CNN
-	1    6300 4650
-	1    0    0    -1
 $EndComp
 $Comp
@@
 F 0 "C2" H 5375 3750 50  0000 L CNN
 F 1 "220u" H 5375 3550 50  0000 L CNN
-F 2 "" H 5350 3650 50  0001 C CNN
+F 2 "Capacitors_ThroughHole:CP_Radial_D7.5mm_P2.50mm" H 5350 3650 50  0001 C CNN
 F 3 "" H 5350 3650 50  0000 C CNN
 	1    5350 3650
@@
 F 0 "R1" V 2630 2500 50  0000 C CNN
 F 1 "1K/2W" V 2450 2500 50  0000 C CNN
-F 2 "" V 2480 2500 50  0001 C CNN
+F 2 "Resistors_ThroughHole:R_Axial_DIN0207_L6.3mm_D2.5mm_P10.16mm_Horizontal" V 2480 2500 50  0001 C CNN
 F 3 "" H 2550 2500 50  0000 C CNN
 	1    2550 2500
@@
 F 0 "P2" H 2050 3050 50  0000 C CNN
 F 1 "PWR" V 2150 2900 50  0000 C CNN
-F 2 "" H 2050 2900 50  0001 C CNN
+F 2 "Socket_Strips:Socket_Strip_Angled_1x02_Pitch2.54mm" H 2050 2900 50  0001 C CNN
 F 3 "" H 2050 2900 50  0000 C CNN
 	1    2050 2900
@@
 F 0 "U3" H 10000 3950 50  0000 C CNN
 F 1 "TRIAC" H 9950 3350 50  0000 C CNN
-F 2 "" H 10250 3600 50  0001 C CNN
+F 2 "Socket_Strips:Socket_Strip_Straight_1x03_Pitch2.54mm" H 10250 3600 50  0001 C CNN
 F 3 "" H 10250 3600 50  0000 C CNN
 	1    10250 3600
@@
 F 0 "R6" V 9430 3800 50  0000 C CNN
 F 1 "56R" V 9350 3800 50  0000 C CNN
-F 2 "" V 9280 3800 50  0001 C CNN
+F 2 "Resistors_SMD:R_1206_HandSoldering" V 9280 3800 50  0001 C CNN
 F 3 "" H 9350 3800 50  0000 C CNN
 	1    9350 3800
@@
 F 0 "P3" H 6100 4300 50  0000 C CNN
 F 1 "NTC probe 10K" V 6200 4150 50  0000 C CNN
-F 2 "" H 6100 4150 50  0001 C CNN
+F 2 "Socket_Strips:Socket_Strip_Straight_1x02_Pitch2.54mm" H 6100 4150 50  0001 C CNN
 F 3 "" H 6100 4150 50  0000 C CNN
 	1    6100 4150
@@
 F 0 "P1" H 2050 2300 50  0000 C CNN
 F 1 "HEATER" V 2150 2150 50  0000 C CNN
-F 2 "" H 2050 2150 50  0001 C CNN
+F 2 "Socket_Strips:Socket_Strip_Angled_1x02_Pitch2.54mm" H 2050 2150 50  0001 C CNN
 F 3 "" H 2050 2150 50  0000 C CNN
 	1    2050 2150
@@
 F 0 "R7" V 10080 4150 50  0000 C CNN
 F 1 "1K" V 10000 4150 50  0000 C CNN
-F 2 "" V 9930 4150 50  0001 C CNN
+F 2 "Resistors_SMD:R_1206_HandSoldering" V 9930 4150 50  0001 C CNN
 F 3 "" H 10000 4150 50  0000 C CNN
 	1    10000 4150
@@
 F 0 "D3" H 8250 3700 50  0000 C CNN
 F 1 "LED" H 8250 3500 50  0000 C CNN
-F 2 "" H 8250 3600 50  0001 C CNN
+F 2 "Socket_Strips:Socket_Strip_Straight_1x02_Pitch2.54mm" H 8250 3600 50  0001 C CNN
 F 3 "" H 8250 3600 50  0000 C CNN
 	1    8250 3600
@@
 Wire Wire Line
 	6300 3700 7100 3700
-Wire Wire Line
-	6300 4200 6300 4650
 $Comp
 L C C1
@@
 F 0 "D1" H 3550 3200 50  0000 C CNN
 F 1 "Diode_Bridge" H 4150 2550 50  0000 C CNN
-F 2 "" H 3800 2900 50  0001 C CNN
+F 2 "Diodes_ThroughHole:Diode_Bridge_15.7x15.7" H 3800 2900 50  0001 C CNN
 F 3 "" H 3800 2900 50  0000 C CNN
 	1    3800 2900
@@
 	5350 3800 5350 4550
 Connection ~ 5350 4550
+Wire Wire Line
+	6300 4200 6300 4550
 $EndSCHEMATC
